Commit message: fix:gazebo spawn issue

File: urdf/environment.xacro (robot description, xacro)
@@ -1,83 +1,81 @@
 <?xml version="1.0" encoding="utf-8"?>
-<!-- This XACRO contains the table and camera models exported from SolidWorks. -->
-<robot xmlns:xacro="http://ros.org/wiki/xacro" name="environment">
-  <!-- abb_table link definition (Root of the environment) -->
-  <link name="abb_table">
-    <inertial>
-      <origin xyz="0.3325 0 -0.561085" rpy="0 0 0" />
-      <mass value="580.907" />
-      <inertia ixx="80.377" ixy="0" ixz="0" iyy="114.089" iyz="0" izz="100.823" />
-    </inertial>
-    <visual>
-      <origin xyz="0 0 0" rpy="0 0 0" />
-      <geometry>
-        <mesh filename="package://assembly_environment/meshes/abb_table.STL" />
-      </geometry>
-      <material name="">
-        <color rgba="0.792 0.820 0.933 1" />
-      </material>
-    </visual>
-    <collision>
-      <origin xyz="0 0 0" rpy="0 0 0" />
-      <geometry>
-        <mesh filename="package://assembly_environment/meshes/abb_table.STL" />
-      </geometry>
-    </collision>
-  </link>
-  <!-- ar4_table link fixed to abb_table -->
-  <link name="ar4_table">
-    <inertial>
-      <origin xyz="-0.429355 0 -0.466079" rpy="0 0 0" />
-      <mass value="173.611" />
-      <inertia ixx="40.833" ixy="0" ixz="-0.418" iyy="53.233" iyz="0" izz="33.728" />
-    </inertial>
-    <visual>
-      <origin xyz="0 0 0" rpy="0 0 0" />
-      <geometry>
-        <mesh filename="package://assembly_environment/meshes/ar4_table.STL" />
-      </geometry>
-      <material name="">
-        <color rgba="0.792 0.820 0.933 1" />
-      </material>
-    </visual>
-    <collision>
-      <origin xyz="0 0 0" rpy="0 0 0" />
-      <geometry>
-        <mesh filename="package://assembly_environment/meshes/ar4_table.STL" />
-      </geometry>
-    </collision>
-  </link>
-  <joint name="ar4_frame" type="fixed">
-    <origin xyz="1.11 0 0.0065" rpy="0 0 3.14159265358979" />
-    <parent link="abb_table" />
-    <child link="ar4_table" />
-  </joint>
-  <!-- camera link fixed to abb_table -->
-  <link name="camera">
-    <inertial>
-      <origin xyz="-0.015 0.115 -0.038" rpy="0 0 0" />
-      <mass value="0.069517" />
-      <inertia ixx="0.000369" ixy="0" ixz="0" iyy="1.347E-05" iyz="0" izz="0.000369" />
-    </inertial>
-    <visual>
-      <origin xyz="0 0 0" rpy="0 0 0" />
-      <geometry>
-        <mesh filename="package://assembly_environment/meshes/camera.STL" />
-      </geometry>
-      <material name="">
-        <color rgba="0.792 0.820 0.933 1" />
-      </material>
-    </visual>
-    <collision>
-      <origin xyz="0 0 0" rpy="0 0 0" />
-      <geometry>
-        <mesh filename="package://assembly_environment/meshes/camera.STL" />
-      </geometry>
-    </collision>
-  </link>
-  <joint name="camera_frame" type="fixed">
-    <origin xyz="0.67 0.01 0.8035" rpy="3.14159265358979 0 1.57079632679489" />
-    <parent link="abb_table" />
-    <child link="camera" />
-  </joint>
+<robot xmlns:xacro="http://ros.org/wiki/xacro">
+  <xacro:macro name="environment">
+    <link name="abb_table">
+      <inertial>
+        <origin xyz="0.3325 0 -0.561085" rpy="0 0 0" />
+        <mass value="580.907" />
+        <inertia ixx="80.377" ixy="0" ixz="0" iyy="114.089" iyz="0" izz="100.823" />
+      </inertial>
+      <visual>
+        <origin xyz="0 0 0" rpy="0 0 0" />
+        <geometry>
+          <mesh filename="file://$(find assembly_environment)/meshes/abb_table.STL" />
+        </geometry>
+        <material name="">
+          <color rgba="0.792 0.820 0.933 1" />
+        </material>
+      </visual>
+      <collision>
+        <origin xyz="0 0 0" rpy="0 0 0" />
+        <geometry>
+          <mesh filename="file://$(find assembly_environment)/meshes/abb_table.STL" />
+        </geometry>
+      </collision>
+    </link>
+    <link name="ar4_table">
+      <inertial>
+        <origin xyz="-0.429355 0 -0.466079" rpy="0 0 0" />
+        <mass value="173.611" />
+        <inertia ixx="40.833" ixy="0" ixz="-0.418" iyy="53.233" iyz="0" izz="33.728" />
+      </inertial>
+      <visual>
+        <origin xyz="0 0 0" rpy="0 0 0" />
+        <geometry>
+          <mesh filename="file://$(find assembly_environment)/meshes/ar4_table.STL" />
+        </geometry>
+        <material name="">
+          <color rgba="0.792 0.820 0.933 1" />
+        </material>
+      </visual>
+      <collision>
+        <origin xyz="0 0 0" rpy="0 0 0" />
+        <geometry>
+          <mesh filename="file://$(find assembly_environment)/meshes/ar4_table.STL" />
+        </geometry>
+      </collision>
+    </link>
+    <joint name="ar4_frame" type="fixed">
+      <origin xyz="1.11 0 0.0065" rpy="0 0 3.14159265358979" />
+      <parent link="abb_table" />
+      <child link="ar4_table" />
+    </joint>
+    <link name="camera">
+      <inertial>
+        <origin xyz="-0.015 0.115 -0.038" rpy="0 0 0" />
+        <mass value="0.069517" />
+        <inertia ixx="0.000369" ixy="0" ixz="0" iyy="1.347E-05" iyz="0" izz="0.000369" />
+      </inertial>
+      <visual>
+        <origin xyz="0 0 0" rpy="0 0 0" />
+        <geometry>
+          <mesh filename="file://$(find assembly_environment)/meshes/camera.STL" />
+        </geometry>
+        <material name="">
+          <color rgba="0.792 0.820 0.933 1" />
+        </material>
+      </visual>
+      <collision>
+        <origin xyz="0 0 0" rpy="0 0 0" />
+        <geometry>
+          <mesh filename="file://$(find assembly_environment)/meshes/camera.STL" />
+        </geometry>
+      </collision>
+    </link>
+    <joint name="camera_frame" type="fixed">
+      <origin xyz="0.67 0.01 0.8035" rpy="3.14159265358979 0 1.57079632679489" />
+      <parent link="abb_table" />
+      <child link="camera" />
+    </joint>
+  </xacro:macro>
 </robot>

Commit message: add new camera made by kareem

File: urdf/environment.xacro (robot description, xacro)
@@ -78,4 +78,37 @@
       <child link="camera" />
     </joint>
+    <link name="camera_optical_frame">
+      <inertial>
+        <mass value="0.001" />
+        <inertia ixx="0.0001" ixy="0" ixz="0" iyy="0.0001" iyz="0" izz="0.0001" />
+      </inertial>
+    </link>
+    <joint name="camera_optical_joint" type="fixed">
+      <origin xyz="0 0 0.025" rpy="3.14 -1.57 -1.57" />
+      <parent link="camera" />
+      <child link="camera_optical_frame" />
+    </joint>
+    <gazebo reference="camera_optical_frame">
+        <sensor name="environment_camera" type="camera">
+        <always_on>true</always_on>
+        <update_rate>30.0</update_rate>
+        <visualize>true</visualize>
+        <topic>/environment_camera/image_raw</topic>
+        <camera>
+            <camera_info_topic>/environment_camera/camera_info</camera_info_topic>
+            <horizontal_fov>1.39626</horizontal_fov>
+            <image>
+            <width>640</width>
+            <height>480</height>
+            <format>R8G8B8</format>
+            </image>
+            <clip>
+            <near>0.02</near>
+            <far>300</far>
+            </clip>
+        </camera>
+        <gz_frame_id>camera_optical_frame</gz_frame_id>
+        </sensor>
+    </gazebo>
   </xacro:macro>
 </robot>

Commit message: change camera to camera optical joint

File: urdf/environment.xacro (robot description, xacro)
@@ -84,6 +84,11 @@
       </inertial>
     </link>
+    <!-- <joint name="camera_optical_joint" type="fixed">
+      <origin xyz="0 0 0.025" rpy="3.14 -1.57 -1.57" />
+      <parent link="camera" />
+      <child link="camera_optical_frame" />
+    </joint> -->
     <joint name="camera_optical_joint" type="fixed">
-      <origin xyz="0 0 0.025" rpy="3.14 -1.57 -1.57" />
+      <origin xyz="0 0 0.025" rpy="1.57079632679 -1.57079632679 0.0" />
       <parent link="camera" />
       <child link="camera_optical_frame" />
