Commit message: add latest changes

File: urdf/environment_hardware.xacro (robot description, xacro)
@@ -78,5 +78,5 @@
       <child link="camera" />
     </joint>
-    <link name="camera_color_optical_frame">
+    <link name="camera_link">
       <inertial>
         <mass value="0.001" />
@@ -84,53 +84,17 @@
       </inertial>
     </link>
-    <joint name="camera_optical_joint" type="fixed">
-      <origin xyz="0 0 0.025" rpy="1.57079632679 -1.57079632679 0.0" />
+    <!-- <joint name="camera_optical_joint" type="fixed">
+      <origin xyz="0 0 0.025" rpy="3.14 -1.57 -1.57" />
       <parent link="camera" />
-      <child link="camera_color_optical_frame" />
+      <child link="camera_link" />
+    </joint> -->
+  <!-- # brick.pose.position.x = brick.pose.position.x - 0.0546
+                # brick.pose.position.y = brick.pose.position.y + 0.674
+                # brick.pose.position.z = 0.769-brick.pose.position.z -->
+    <joint name="camera_color_optical_frame" type="fixed">
+      <origin xyz="0.674 -0.0546 0.769" rpy="3.14 1.57 0.0" />
+      <parent link="abb_table" />
+      <child link="camera_link" />
     </joint>
-     <!-- <joint name="camera_optical_joint" type="fixed">
-      <origin xyz="0 0 0.025" rpy="0.0 0.0 0.0" />
-      <parent link="camera" />
-      <child link="camera_color_optical_frame" />
-    </joint> -->
-    <gazebo reference="camera_color_optical_frame">
-    <sensor name="env_cam_rgb" type="camera">
-        <always_on>true</always_on>
-        <update_rate>30.0</update_rate>
-        <visualize>false</visualize>
-        <topic>/environment_camera/image_raw</topic> <camera>
-            <camera_info_topic>/environment_camera/camera_info</camera_info_topic>
-            <horizontal_fov>1.518436</horizontal_fov>
-            <image>
-                <width>1280</width>
-                <height>720</height>
-                <format>R8G8B8</format>
-            </image>
-            <clip>
-                <near>0.02</near>
-                <far>300</far>
-            </clip>
-        </camera>
-        <gz_frame_id>camera_color_optical_frame</gz_frame_id>
-    </sensor>
-    <sensor name="env_cam_depth" type="depth_camera">
-        <always_on>true</always_on>
-        <update_rate>30.0</update_rate>
-        <visualize>true</visualize>
-        <topic>/environment_camera/depth_image</topic> <camera>
-            <horizontal_fov>1.518436</horizontal_fov>
-            <image>
-                <width>1280</width>
-                <height>720</height>
-                <format>R_FLOAT32</format>
-            </image>
-            <clip>
-                <near>0.02</near>
-                <far>300</far>
-            </clip>
-        </camera>
-        <gz_frame_id>camera_color_optical_frame</gz_frame_id>
-    </sensor>
-  </gazebo>
-  </xacro:macro>
+    </xacro:macro>
 </robot>
